File: boards/HeyListen/HeyListen.kicad_pcb (KiCad board)
At the start: 2 copper layers, 40.1 x 41.9 mm, 13 parts, among them J1 Conn_01x04, J2 Conn_01x04, J3 Conn_01x04, J4 Conn_01x02, J5 Conn_01x02, J6 Conn_01x03, Q1 2N3904, U1 ESP-01, U2 ESP-01, U3 ESP-01

Commit message: Fixed a disconnected GND
Routing:
- net /V3P3: track 72.6 -> 73.2 mm, vias 0 -> 2
Other:
- rule via_min_size: 0.4 -> 0.2
